File: kicad/IRLED1.sch (KiCad schematic (older format))
At the start: 10 parts

Commit message: more work on the schematic
Parts:
- added C? (x3): C, symbol C
- added C? (x3): CP1, symbol CP1
- added D?: LED, symbol LED
- added J?: CONN_01X06, symbol CONN_01X06
- added J?: POWER, symbol CONN_01X02
- added Q?: 2N7002, symbol 2N7002
- added R?: R, symbol R
- added R? (x3): 10k, symbol R
- added SW?: RST, symbol SW_PUSH_SMALL
Connections:
- net VBAT: now reaches U?.1 (INPUT)
- net VBAT: now also U?.1 (VDD), U?.~ (VIN), C?.1, C?.1, C?.1, C?.1, J?.1 (P1)
- net +3.3V: now reaches U?.3 (OUT)
- net +3.3V: now also J?.2 (P2), R?.2, R?.2
- net DIM: now reaches U?.4 (ADJ)
- net DIM: now also C?.1, R?.2
- net at U?.3 (GND): now also U?.8 (GND), U?.8 (VSS), C?.2, C?.2, C?.2, C?.2
- net at U?.2 (RA5): now also R?.1
- net ~MCLR: now reaches U?.3 (~MLCR~/VPP/RA3)
- net ~MCLR: now also C?.1, J?.1 (P1), R?.1, SW?.2
- net PGC: now reaches U?.6 (ICSPCLK/RA1)
- net PGC: now also J?.5 (P5)
- net IND: now reaches U?.7 (ICSPDAT/RA0)
- net IND: now also J?.4 (P4), R?.2
- new net: Q?.1 (G), R?.1
- new net: D?.1 (K), Q?.3 (D)
- new net: D?.2 (A), R?.1
- new net GND: C?.2, C?.2, J?.2 (P2), J?.3 (P3), Q?.2 (S), SW?.1
- no-connect marks 0 -> 1
Other:
- moved on the sheet: D?, R?, U?, U?B

Commit message: more work on the schematic
Parts:
- added Q?: 2N7002, symbol 2N7002
- added Q?: FDN340P, symbol FDN340P
- added R? (x2): 10k, symbol R
- C?: value C -> DNF
- R?: value R -> DNF
Connections:
- net +3.3V: now also C?.1, U?.1 (VDD)
- net VBAT: now also Q?.2 (D), R?.2; no longer C?.1, C?.1, U?.1 (VDD), U?.~ (VIN)
- net at C?.2, C?.2, C?.2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: now also Q?.2 (S), R?.1
- new net: C?.1, Q?.3 (S), U?.~ (VIN)
- new net: Q?.1 (G), Q?.3 (D), R?.1
- new net LED_EN: Q?.1 (G), R?.2
Other:
- moved on the sheet: C?, U?B

Commit message: more work on schematic
Parts:
- removed D?: LD4, symbol Led_Small
- removed U?: 78M33, symbol 78M33
- added J2: LED, bjh-kicad-connector-fp:HEAD-1row-2.54mm-2way, symbol CONN_01X02
- added R3: 10k, Resistors_SMD:R_0805, symbol R
- added SW2: MODE, bjh-kicad-switches-fp:PushButton-OMRON-B3FS, symbol SW_PUSH_SMALL
- added U2: 78M33, TO_SOT_Packages_SMD:SOT-223, symbol 78M33
- C1, C2, C3, C4, C5, C6, C7: renamed from C?; footprint (none) -> Capacitors_SMD:C_0805
- D1: renamed from D?; footprint (none) -> Diodes_SMD:SMA_Standard
- D2: renamed from D?; footprint (none) -> LEDs:LED_1206
- J1: renamed from J?; footprint (none) -> bjh-kicad-connector-fp:HEAD-1row-2.54mm-2way
- J3: renamed from J?; footprint (none) -> bjh-kicad-connector-fp:HEAD-1row-2.54mm-6way
- Q1, Q2, Q3: renamed from Q?; footprint (none) -> TO_SOT_Packages_SMD:SOT-23
- R1, R2, R4, R5, R7, R8: renamed from R?; footprint (none) -> Resistors_SMD:R_0805
- R6: renamed from R?; footprint (none) -> Resistors_SMD:R_1210
- SW1: renamed from SW?; footprint (none) -> bjh-kicad-switches-fp:PushButton-OMRON-B3FS
- U1: renamed from U?; footprint (none) -> SMD_Packages:SOIC-8-N
- U3: renamed from U?; footprint (none) -> TO_SOT_Packages_SMD:SOT-23-5
- gave numbers to parts that had none: 1
Connections:
- net +3.3V: now also R3.2, U2.3 (OUT)
- net GND: now also SW2.1
- net LED_EN: now also U1.3 (~MLCR~/VPP/RA3)
- net VBAT: now also U2.1 (INPUT)
- net A: now reaches C6.1, R6.2, U3.2 (SENSE)
- net A: now also J2.1 (P1)
- net VBAT_SW: now reaches C5.1, Q2.3 (S), U3.~ (VIN)
- net VBAT_SW: now also D1.1 (K), R6.1
- net K: now reaches C6.2, L1.1
- net K: now also J2.2 (P2)
- net MODE: now reaches U1.5 (RA2)
- net MODE: now also R3.1, SW2.2
Other:
- moved on the sheet: C5, C6, C7, D1, D2, J3, L1, Q1, Q2, Q3, R4, R5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

Commit message: Version 1 schematic complete including PCB design
Parts:
- removed C3: C, Capacitors_SMD:C_0805, symbol C
- removed J1: POWER, bjh-kicad-connector-fp:HEAD-1row-2.54mm-2way, symbol CONN_01X02
- removed J2: LED, bjh-kicad-connector-fp:HEAD-1row-2.54mm-2way, symbol CONN_01X02
- removed J3: CONN_01X06, bjh-kicad-connector-fp:HEAD-1row-2.54mm-6way, symbol CONN_01X06
- removed SW1: RST, bjh-kicad-switches-fp:PushButton-OMRON-B3FS, symbol SW_PUSH_SMALL
- removed U3: RT8471_BJH, TO_SOT_Packages_SMD:SOT-23-5, symbol RT8471_BJH
- added J1: POWER, bjh-kicad-connector-fp:MATE-N-LOK-RIGHT-ANGLE-2WAY_smt_2-1445057-2, symbol CONN_01X03
- added J2: LED, bjh-kicad-connector-fp:MATE-N-LOK-RIGHT-ANGLE-2WAY_smt_2-1445057-2, symbol CONN_01X03
- added R9: 0R, Resistors_SMD:R_1206, symbol R
- added TP1: PWM, bjh-kicad-connector-fp:TP_smt, symbol CONN_01X01
- added U3: RT8471_MSOP-8, bjh-kicad-ic-fp:MSOP-8a, symbol RT8471_MSOP-8
- C1: value CP1 -> 0.33u
- C2: value DNF -> DNP
- C4: value CP1 -> 0.1u
- C5: value CP1 -> 4u7
- C6: value 1uF -> DNP
- L1: footprint (none) -> bjh-kicad-rcld-fp:Inductor_SRN6045
- R2: value DNF -> 0R
- SW2: footprint bjh-kicad-switches-fp:PushButton-OMRON-B3FS -> Buttons_Switches_SMD:SW_SPST_KMR2
Connections:
- net +3.3V: now also C4.1
- net A: now also J2.1 (P1), U3.1 (SENSE)
- net DIM: now also R9.1, R9.2, TP1.1 (P1), U3.4 (ADJ)
- net GND: now also C1.2, C4.2, C5.2, C7.2, Q1.2 (S), R4.1, U1.8 (VSS), U2.2 (COM), U2.4 (COM), J1.2 (P2), J1.3 (P3), U3.2 (GND), U3.3 (GND), U3.9 (GND)
- net K: now also J2.2 (P2)
- net VBAT: now also J1.1 (P1); no longer C4.1
- net VBAT_SW: now also U3.8 (VIN)
- net at D1.2 (A), L1.2: now also U3.5 (LX), U3.6 (LX)
Other:
- moved on the sheet: C4
