File: kicad/IRLED1.sch (KiCad schematic (older format))
At the start: 29 parts, among them J1 POWER, J2 LED, J3 CONN_01X06, Q1 2N7002, Q2 FDN340P, Q3 2N7002, SW1 RST, SW2 MODE, U1 PIC-12F1822, U2 78M33, U3 RT8471_BJH

Commit message: Working towards circular PCB
Parts:
- added D3: D, symbol D
- U2: symbol 78M33 -> 78M33-RESCUE-IRLED1
Connections:
- net +3.3V: now also D3.2 (A); no longer C1.1, C4.1, Q2.2 (D), R5.2, U2.1 (INPUT)
- new net: C1.1, C4.1, D3.1 (K), Q2.2 (D), R5.2, U2.1 (INPUT)
Changed lines of the file:
@@
 EESchema Schematic File Version 2
+LIBS:IRLED1-rescue
 LIBS:power
 LIBS:device
@@
 $EndComp
 $Comp
-L VBAT_BJH #PWR07
+L VBAT_BJH-RESCUE-IRLED1 #PWR07
 U 1 1 58DAF598
 P 10600 800
@@
 $EndComp
 $Comp
-L VBAT_BJH #PWR08
+L VBAT_BJH-RESCUE-IRLED1 #PWR08
 U 1 1 58DAF815
-P 650 800
-F 0 "#PWR08" H 650 990 20  0001 C CNN
-F 1 "VBAT_BJH" H 650 990 51  0001 C CNN
-F 2 "" H 650 800 60  0001 C CNN
-F 3 "" H 650 800 60  0001 C CNN
-F 4 "VBAT" H 650 1000 60  0000 C CNB "NAME"
-	1    650  800
+P 600 800
+F 0 "#PWR08" H 600 990 20  0001 C CNN
+F 1 "VBAT_BJH" H 600 990 51  0001 C CNN
+F 2 "" H 600 800 60  0001 C CNN
+F 3 "" H 600 800 60  0001 C CNN
+F 4 "VBAT" H 600 1000 60  0000 C CNB "NAME"
+	1    600  800
 	1    0    0    -1
 $EndComp
@@
 $EndComp
 $Comp
-L VBAT_SW_BJH #PWR013
+L VBAT_SW_BJH-RESCUE-IRLED1 #PWR013
 U 1 1 58DF9B60
 P 5250 800
@@
 $EndComp
 $Comp
-L VBAT_SW_BJH #PWR014
+L VBAT_SW_BJH-RESCUE-IRLED1 #PWR014
 U 1 1 58DF9C5C
 P 6100 3050
@@
 K
 $Comp
-L VBAT_BJH #PWR016
+L VBAT_BJH-RESCUE-IRLED1 #PWR016
 U 1 1 58E01DC4
 P -6850 -5000
@@
 $EndComp
 $Comp
-L VBAT_SW_BJH #PWR018
+L VBAT_SW_BJH-RESCUE-IRLED1 #PWR018
 U 1 1 58E01E98
 P -6200 -5000
@@
 IND
 $Comp
-L 78M33 U2
+L 78M33-RESCUE-IRLED1 U2
 U 1 1 58E0412D
 P 1500 1750
@@
 	10600 850  10600 1050
 Wire Wire Line
-	650  850  650  1100
-Wire Wire Line
 	1500 1100 1500 1200
 Wire Wire Line
@@
 Connection ~ 5350 2400
 Wire Wire Line
-	4000 1200 4000 1100
+	4000 1100 4000 1200
 Wire Wire Line
 	4000 1500 4000 1650
@@
 Connection ~ 6100 3300
 Wire Wire Line
-	650  1100 4150 1100
-Wire Wire Line
 	2200 850  2200 1750
 Connection ~ 2400 1100
@@
 	5500 4100 5500 4150
 Connection ~ 5500 4150
+$Comp
+L D D3
+U 1 1 596E39CB
+P 750 1100
+F 0 "D3" H 750 1200 50  0000 C CNN
+F 1 "D" H 750 1000 50  0000 C CNN
+F 2 "" H 750 1100 50  0000 C CNN
+F 3 "" H 750 1100 50  0000 C CNN
+	1    750  1100
+	-1   0    0    1
+$EndComp
+Wire Wire Line
+	600  850  600  1100
+Wire Wire Line
+	900  1100 4150 1100
 $EndSCHEMATC
